Commit message: week 4 code update

File: legged_dora2_him/src/legged_rl_encoder/legged_robot/dora2/legged_dora2_description/urdf/dora2 copy_erect.urdf (robot description, URDF)
Before this commit: robot dora2, 22 links, 21 joints
Joints:
- joint leg_r1_joint: origin xyz=-0.0792 -0.09002 -0.085 rpy=0 0 0 -> xyz=-0.0792 -0.08998 -0.085 rpy=0 0 0

File: legged_dora2_him/src/legged_rl_encoder/legged_robot/dora2/legged_dora2_description/urdf/dora2_6_erect.urdf (robot description, URDF)
Before this commit: robot Dora2, 21 links, 20 joints
Links:
- link l_leg_ankle_pitch_Link: mass 0.0899541151447192 -> 0.089954
- link l_leg_ankle_roll_Link: mass 0.442108383473458 -> 0.44211
- link l_leg_knee_Link: mass 1.34567623230749 -> 1.3457
- link r_arm_shoulder_pitch_Link: mass 0.474849451126101 -> 0.47485
- link r_arm_shoulder_roll_Link: mass 0.369997409547943 -> 0.369997353872883
- link r_arm_shoulder_yaw_Link: mass 0.38568 -> 0.385684351005629
Joints:
- joint l_arm_elbow_joint: limit lower=-1.5 upper=1.5 effort=100 velocity=12 -> lower=-1.5 upper=1.5 effort=36 velocity=12
- joint l_arm_shoulder_pitch_joint: limit lower=-2 upper=2 effort=100 velocity=12 -> lower=-2 upper=2 effort=36 velocity=12
- joint l_arm_shoulder_roll_joint: limit lower=0 upper=3 effort=100 velocity=12 -> lower=0 upper=3 effort=36 velocity=12
- joint l_arm_shoulder_yaw_joint: limit lower=-2 upper=2 effort=100 velocity=12 -> lower=-2 upper=2 effort=36 velocity=12
- joint l_leg_hip_pitch_joint: limit lower=-1.12 upper=0.88 effort=150 velocity=12 -> lower=-1.12 upper=0.88 effort=150 velocity=100
- joint r_arm_elbow_joint: limit lower=-1.5 upper=1.5 effort=100 velocity=12 -> lower=-1.5 upper=1.5 effort=36 velocity=12
- joint r_arm_shoulder_pitch_joint: limit lower=-2 upper=2 effort=100 velocity=12 -> lower=-2 upper=2 effort=36 velocity=12
- joint r_arm_shoulder_roll_joint: limit lower=-3 upper=0 effort=100 velocity=12 -> lower=-3 upper=0 effort=36 velocity=12
- joint r_arm_shoulder_yaw_joint: limit lower=-2 upper=2 effort=100 velocity=12 -> lower=-2 upper=2 effort=36 velocity=12
- joint r_leg_hip_roll_joint: origin xyz=-0.0792 -0.08998 -0.085 rpy=0 0 0 -> xyz=-0.0792 -0.09002 -0.085 rpy=0 0 0
- joint r_leg_knee_joint: origin xyz=0 -0.0327 -0.27 rpy=0 0.4 0 -> xyz=0 -0.032659 -0.27 rpy=0 0.4 0
